File: kicad/som_fpga.kicad_pcb (KiCad board)
At the start: 4 copper layers, 60 x 50 mm, 88 parts, among them J1 Conn_01x02_Pin, J2 Conn_02x20_Odd_Even, J3 Conn_02x20_Odd_Even, J4 Conn_02x20_Odd_Even, U1 XC7A35T-FGG484, U2 TLV62565DBVR, U3 TLV62565DBVR, U4 TLV62565DBVR, U5 MX25L12833F, U6 cp_logo25mm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

Commit message: cp_som_Altium imported
Parts:
- removed U6: cp_logo25mm, cplogo:logo25mm
Other:
- board text added: "ENG/ESLAM FAYAD"
